File: Zenith_ZA-M5.kicad_sch (KiCad schematic)
At the start: 68 parts

Commit message: Fix a description
Parts:
- C311?: Notes (none) -> Label not visible - near CN303 pins 9 & 10
- C312: Notes (none) -> Value not fully visible

Commit message: Remove a ? from a capacitor value I've removed the cap so I can now see it's the value I thought it was!
Parts:
- C312: value 10V100uF? -> 10V100uF
Changed lines of the file:
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@@
 			)
 		)
-		(property "Value" "10V100uF?"
+		(property "Value" "10V100uF"
 			(at 71.12 155.194 90)
 			(effects
